File: Pi-Expansion/Pi-Expansion.sch (KiCad schematic (older format))
At the start: 12 parts, among them J1 RPi_GPIO, J2 SMA_H, P1 BATT, Q1 IRLML6344TRPBF, U1 A2200-A, U2 SPX2920U-5.0

Commit message: Rejigged librarys abit to be less random, made sure to use submodules instead of local copys. Also did first draft of pcb layout
Parts:
- J2: footprint SMA_H -> Universal:SMA_H
- Q1: footprint FT:SOT23-3 -> FT:SOT23_FET
Changed lines of the file:
@@
 LIBS:contrib
 LIBS:valves
+LIBS:Universal
 LIBS:a2200-a
 LIBS:RPi_Hat-cache
-LIBS:Universal
 LIBS:Pi-Expansion-cache
 EELAYER 25 0
@@
 F 0 "J2" H 4850 2250 60  0000 C CNN
 F 1 "SMA_H" H 4750 2400 60  0001 C CNN
-F 2 "SMA_H" H 4750 2500 60  0001 C CNN
+F 2 "Universal:SMA_H" H 4750 2500 60  0001 C CNN
 F 3 "" H 4975 2115 60  0000 C CNN
 F 4 "Digi-Key" H 4750 2950 60  0001 C CNN "Vendor"
@@
 F 0 "Q1" V 9410 1320 60  0000 R CNN
 F 1 "IRLML6344TRPBF" V 9560 900 60  0000 R CNN
-F 2 "FT:SOT23-3" H 9500 1150 60  0001 C CNN
+F 2 "FT:SOT23_FET" H 9500 1150 60  0001 C CNN
 F 3 "" H 9500 1150 60  0000 C CNN
 	1    9500 1150
